Commit message: remove debug urdf , adjust urdf from x -> y to be better in line with initialization

File: assets/urdf/assembly/kinova3_robotiq_2f_85/kinova_gen3_robotiq_2f_85_left.urdf (robot description, URDF)
Before this commit: robot gen3, 18 links, 17 joints
Joints:
- joint base_joint: origin xyz=-0.5 0 0 rpy=0 0 0 -> xyz=0 -0.5 0 rpy=0 0 0

File: assets/urdf/assembly/kinova3_robotiq_2f_85/kinova_gen3_robotiq_2f_85_right.urdf (robot description, URDF)
Before this commit: robot gen3, 18 links, 17 joints
Joints:
- joint base_joint: origin xyz=0.5 0 0 rpy=0 0 0 -> xyz=0 0.5 0 rpy=0 0 0
