Commit message: urdf fixes

File: assets/urdf/assembly/wxai_base/wxai_arm_left.urdf (robot description, URDF)
Before this commit: robot wxai, 12 links, 11 joints
Links:
- link base_link: geometry collision mesh filename=../../arms/wxai_base_arm/collision/base_link.obj; visual mesh filename=../../arms/wxai_base_arm/visual/base_link.stl
- link carriage_left: geometry collision mesh filename=../../arms/wxai_base_arm/collision/carriage_left.obj; visual mesh filename=../../arms/wxai_base_arm/visual/carriage_left.stl
- link carriage_right: geometry collision mesh filename=../../arms/wxai_base_arm/collision/carriage_right.obj; visual mesh filename=../../arms/wxai_base_arm/visual/carriage_right.stl
- link gripper_left: geometry collision mesh filename=../../arms/wxai_base_arm/collision/gripper_left.obj; visual mesh filename=../../arms/wxai_base_arm/visual/gripper_left.stl
- link gripper_right: geometry collision mesh filename=../../arms/wxai_base_arm/collision/gripper_right.obj; visual mesh filename=../../arms/wxai_base_arm/visual/gripper_right.stl
- link link_1: geometry collision mesh filename=../../arms/wxai_base_arm/collision/link_1.obj; visual mesh filename=../../arms/wxai_base_arm/visual/link_1.stl
- link link_2: geometry collision mesh filename=../../arms/wxai_base_arm/collision/link_2.obj; visual mesh filename=../../arms/wxai_base_arm/visual/link_2.stl
- link link_3: geometry collision mesh filename=../../arms/wxai_base_arm/collision/link_3.obj; visual mesh filename=../../arms/wxai_base_arm/visual/link_3.stl
- link link_4: geometry collision mesh filename=../../arms/wxai_base_arm/collision/link_4.obj; visual mesh filename=../../arms/wxai_base_arm/visual/link_4.stl
- link link_5: geometry collision mesh filename=../../arms/wxai_base_arm/collision/link_5.obj; visual mesh filename=../../arms/wxai_base_arm/visual/link_5.stl
- link link_6: geometry collision mesh filename=../../arms/wxai_base_arm/collision/link_6.obj; visual mesh filename=../../arms/wxai_base_arm/visual/link_6.stl
